File: schematics/rp2040_black_vga/rp2040_black_vga.kicad_sch (KiCad schematic)
At the start: 42 parts, among them J1 Jack-DC, J2 Conn_01x02, J2B1 DE15_Socket_HighDensity_Mount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, J3 Conn_02x06_Top_Bottom, J4 Mini-DIN-6, J5 Conn_02x20_Odd_Even, J6 DE9_Pins, J7 DE9_Pins, J8 Audio OUT, J8B1 OUT_A, U1 YD-RP2040 TypeC Black Clone

Commit message: audio-in added
Parts:
- added C11, C12: 100n, Capacitor_THT:C_Disc_D5.0mm_W2.5mm_P2.50mm, symbol Device:C
- added D4: 4148, symbol Device:D
- added J9: Audio IN, Connector_Audio:Jack_3.5mm_CUI_SJ1-3535NG_Horizontal, symbol Connector:AudioJack3_SwitchTR
- added J9B1: IN_A, Connector_PinHeader_2.54mm:PinHeader_1x03_P2.54mm_Vertical, symbol Connector_Generic:Conn_01x02
- added NT1, NT2, NT3, NT4, NT5, NT6: NetTie_2, symbol Device:NetTie_2
- added Q1, Q2: S9014, symbol Device:Q_NPN
- added R29, R30, R32: 10K, _my_Resistors:R_Axial_DIN0207_L6.3mm_D2.2mm_P10.16mm_Horizontal, symbol Device:R
- added R31: 1K, _my_Resistors:R_Axial_DIN0207_L6.3mm_D2.2mm_P10.16mm_Horizontal, symbol Device:R
- added R33: 100R, _my_Resistors:R_Axial_DIN0207_L6.3mm_D2.2mm_P10.16mm_Horizontal, symbol Device:R
- C10, C5, C7, C8, C9: footprint LIBS:R_0805_PLUS -> Capacitor_THT:C_Disc_D5.0mm_W2.5mm_P2.50mm
- R1, R3, R5: value R_Small -> 1K; footprint (none) -> _my_Resistors:R_Axial_DIN0207_L6.3mm_D2.2mm_P10.16mm_Horizontal
- R10, R11, R12, R9: footprint (none) -> _my_Resistors:R_Axial_DIN0207_L6.3mm_D2.2mm_P10.16mm_Horizontal
- R2, R4, R6: value R_Small -> 330R; footprint (none) -> _my_Resistors:R_Axial_DIN0207_L6.3mm_D2.2mm_P10.16mm_Horizontal
- R21, R25: value 1k -> 1K; footprint LIBS:R_0805_PLUS -> _my_Resistors:R_Axial_DIN0207_L6.3mm_D2.2mm_P10.16mm_Horizontal
- R22, R26, R27, R28: footprint LIBS:R_0805_PLUS -> _my_Resistors:R_Axial_DIN0207_L6.3mm_D2.2mm_P10.16mm_Horizontal
- R23, R24: value 2k -> 2K; footprint LIBS:R_0805_PLUS -> _my_Resistors:R_Axial_DIN0207_L6.3mm_D2.2mm_P10.16mm_Horizontal
- R7, R8: value R_Small -> 100R; footprint (none) -> _my_Resistors:R_Axial_DIN0207_L6.3mm_D2.2mm_P10.16mm_Horizontal
Connections:
- net GP_14 is gone; now on net CLOCK: J5.2 (Pin_2)
- net GP_15 is gone; now on net LATCH: J5.4 (Pin_4)
- net GP_16 is gone; now on net DATA1: J5.6 (Pin_6)
- net GP_29_VREF is gone; now on net GP_29: J5.28 (Pin_28)
- net +3V3: now also C12.1, R30.1, R31.1
- net +5V: no longer J5.38 (Pin_38)
- net +5V_VOUT: now also J5.38 (Pin_38)
- net BEEP_OUT: now also NT4.1; no longer J5.26 (Pin_26)
- net DATA2: now also J5.8 (Pin_8)
- net GND: now also C12.2, J9.S, J9B1.2 (Pin_2), Q1.E, Q2.E, R33.2
- net GP_0: now also NT6.2; no longer D2.1 (K), J5.31 (Pin_31), R11.2
- net GP_1: now also NT5.2; no longer D3.1 (K), J5.29 (Pin_29), R12.2
- net GP_17: no longer J5.8 (Pin_8)
- net GP_18: now also U1.24 (GP18)
- net GP_19: now also U1.25 (GP19)
- net GP_20: now also U1.26 (GP20)
- net GP_21: now also U1.27 (GP21)
- net GP_22: now also U1.29 (GP22), NT1.2
- net GP_26: now also NT2.2; no longer J5.21 (Pin_21), R25.2
- net GP_27: now also NT3.2; no longer J5.23 (Pin_23), R21.2
- net LOAD_IN_D: now also NT1.1, Q2.C, R31.2
- net RUN: now also U1.30 (RUN)
- net GP_29: now reaches U1.35 (GP29)
- new net: D4.2 (A), Q1.C, R29.1, R30.2
- new net: Q2.B, R29.2
- new net: D4.1 (K), Q1.B, R32.2
- new net: C11.1, R32.1
- new net GP_28: J5.26 (Pin_26), NT4.2
- new net LEFT_OUT: J5.23 (Pin_23), NT3.1, R21.2
- new net LOAD_IN_L: C11.2, J9.T, J9B1.1 (Pin_1), R33.1
- new net PS/2_CLK_3V: D2.1 (K), J5.31 (Pin_31), NT6.1, R11.2
- new net PS/2_DATA_3V: D3.1 (K), J5.29 (Pin_29), NT5.1, R12.2
- new net RIGHT_OUT: J5.21 (Pin_21), NT2.1, R25.2
- no-connect marks 46 -> 42
Other:
- note added: "Audio-In Interface"
- note added: "Audio-Out Interface"
- note added: "External Connector"
- note added: "GP_14"
- note added: "GP_15"
- note added: "GP_16"
- note added: "GP_17"
- company: (none) -> Alex Snigir
- title: (none) -> Murmulator on RP2040 (black clone) module with VGA
- moved on the sheet: C10, C4, C5, C6, C7, J2B1, J3, J5, J8, J8B1, R1, R2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

Commit message: update schematics
Parts:
- removed J8: Audio OUT, Connector_Audio:Jack_3.5mm_CUI_SJ1-3535NG_Horizontal, symbol Connector:AudioJack3_SwitchTR
- removed J9: Audio IN, Connector_Audio:Jack_3.5mm_CUI_SJ1-3535NG_Horizontal, symbol Connector:AudioJack3_SwitchTR
- added C15, C17, C20: 100nF, Capacitor_THT:C_Disc_D5.0mm_W2.5mm_P2.50mm, symbol Device:C_Small
- added C16, C18: 100uF, Capacitor_THT:CP_Radial_D6.3mm_P2.50mm, symbol Device:C_Polarized
- added C19: 470uF, Capacitor_THT:CP_Radial_D8.0mm_P2.50mm, symbol Device:C_Polarized
- added J10, J11: Conn_01x02, Connector_JST:JST_XH_S2B-XH-A_1x02_P2.50mm_Horizontal, symbol Connector_Generic:Conn_01x02
- added J8: Audio OUT, Connector_Audio:Jack_3.5mm_CUI_SJ1-3525N_Horizontal, symbol Connector_Audio:AudioJack3_SwitchTR
- added J9: Audio IN, Connector_Audio:Jack_3.5mm_CUI_SJ1-3525N_Horizontal, symbol Connector_Audio:AudioJack3_SwitchTR
- added NT7: NetTie_2, Connector_PinHeader_2.54mm:PinHeader_1x02_P2.54mm_Vertical, symbol Device:NetTie_2
- added SW1: RESET, Button_Switch_THT:SW_Tactile_SKHH_Angled, symbol Switch:SW_Push
- C10, C11, C12, C8, C9: value 100n -> 100nF
- C4, C6: value 10u -> 10uF
- C5, C7: value 10n -> 10nF
- D1: footprint Diode_THT:D_DO-41_SOD81_P10.16mm_Horizontal -> Diode_THT:D_DO-41_SOD81_P7.62mm_Horizontal
- D2, D3: footprint (none) -> Diode_THT:D_DO-41_SOD81_P7.62mm_Horizontal
- D4: footprint (none) -> Diode_THT:D_DO-35_SOD27_P7.62mm_Horizontal
- J2B1: value DE15_Socket_HighDensity_MountingHoles -> DE15_Socket
- J3: footprint (none) -> Connector_PinHeader_1.00mm:PinHeader_2x06_P1.00mm_Vertical
- J4: footprint (none) -> _my_Connectors:Connector_Mini-DIN_Female_6Pin_2rows
- J6, J7: footprint (none) -> _my_Connectors:DB9_PinHeader_1x05_P2.54mm_Pins_2,3,4,6,8
- Q1, Q2: footprint (none) -> _my_Transistors:TO-92_Inline_Wide_S9014
- U2: footprint (none) -> Connector_PinHeader_2.54mm:PinHeader_1x06_P2.54mm_Vertical
Connections:
- net +3V3: now also C15.1, C16.1, J10.2 (Pin_2)
- net +5V_VOUT: now also J5.39 (Pin_39), J5.40 (Pin_40), C17.1, C18.1, J11.2 (Pin_2); no longer D1.1 (K), J5.38 (Pin_38)
- net GND: now also C15.2, C16.2, C17.2, C18.2, C19.2, C20.2, J10.1 (Pin_1), J11.1 (Pin_1), J8.S, J9.S, SW1.2; no longer J5.35 (Pin_35)
- net L: now also J8.T
- net LOAD_IN_L: now also J9.T
- net R: now also J8.R
- net RUN: now also NT7.1, SW1.1; no longer J5.36 (Pin_36)
- net GP_23: now reaches U1.37 (GP23)
- net GP_23: now also J5.36 (Pin_36)
- net +5V renamed +5V_RAW
- net +5V_RAW: now also C19.1; no longer J5.39 (Pin_39), J5.40 (Pin_40), U1.39 (Vin)
- new net +5V_IN: C20.1, D1.1 (K), J5.38 (Pin_38), U1.39 (Vin)
- new net RST: J5.35 (Pin_35), NT7.2
- no-connect marks 42 -> 41
Other:
- note added: "ADC_VREF"
- note added: "Power 3V Out"
- note added: "Power 5V Out"
- note added: "RAW Power Out"
- note added: "RAW Power Out connected to +5V_RAW to prevent powering through Vout/VBUS pin 40 of MC"
- note removed: "Power Out"
- moved on the sheet: C11, C12, C4, C5, C6, C7, D1, D4, J8B1, J9B1, Q1, Q2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

Commit message: 3d models, doc and pcb update
Parts:
- removed U2: (no value), Connector_PinHeader_2.54mm:PinHeader_1x06_P2.54mm_Vertical, symbol _my_Generic_components:MicroSD_Module
- added J12: (no value), _my_Generic_Modules:USB_Micro_Module_15x13.5mm, symbol _my_Generic_Modules:USB_Micro_Module
- added J13: Conn_01x03, Connector_PinHeader_2.54mm:PinHeader_1x03_P2.54mm_Vertical, symbol Connector_Generic:Conn_01x03
- added J14: Conn_01x02, Connector_PinHeader_2.54mm:PinHeader_1x02_P2.54mm_Vertical, symbol Connector_Generic:Conn_01x02
- added J15: (no value), _my_Generic_Modules:MicroSD_Module_41.5x24.5mm, symbol _my_Generic_Modules:MicroSD_Module
- added J16: Conn_01x02, Connector_JST:JST_XH_S2B-XH-A_1x02_P2.50mm_Horizontal, symbol Connector_Generic:Conn_01x02
- added NT8: NetTie_2, symbol Device:NetTie_2
- C19: footprint Capacitor_THT:CP_Radial_D8.0mm_P2.50mm -> Capacitor_THT:CP_Radial_Tantal_D8.0mm_P5.00mm
- C5, C7: footprint Capacitor_THT:C_Disc_D5.0mm_W2.5mm_P2.50mm -> Capacitor_THT:C_Disc_D5.0mm_W2.5mm_P5.00mm
- J1: footprint Connector_PinHeader_2.54mm:PinHeader_1x02_P2.54mm_Vertical -> Connector_BarrelJack:BarrelJack_Horizontal
- J10: footprint Connector_JST:JST_XH_S2B-XH-A_1x02_P2.50mm_Horizontal -> _my_Connectors:JST_XH_S2B_1x02_P2.50mm_Horizontal
- J11: footprint Connector_JST:JST_XH_S2B-XH-A_1x02_P2.50mm_Horizontal -> (none)
- J2B1: footprint (none) -> _my_Generic_Modules:VGA_DR15P_Module
- J3: footprint Connector_PinHeader_1.00mm:PinHeader_2x06_P1.00mm_Vertical -> (none)
- J6, J7: footprint _my_Connectors:DB9_PinHeader_1x05_P2.54mm_Pins_2,3,4,6,8 -> _my_Connectors:DB9_PinHeader_1x05_P2.54mm_Pins_4,3,8,6,2
- J9B1: footprint Connector_PinHeader_2.54mm:PinHeader_1x03_P2.54mm_Vertical -> Connector_PinHeader_2.54mm:PinHeader_1x02_P2.54mm_Vertical
- R10, R11, R12, R29, R30, R31, R32, R33, R9: footprint _my_Resistors:R_Axial_DIN0207_L6.3mm_D2.2mm_P10.16mm_Horizontal -> Resistor_THT:R_Axial_DIN0207_L6.3mm_D2.5mm_P7.62mm_Horizontal
- SW1: footprint Button_Switch_THT:SW_Tactile_SKHH_Angled -> _my_Custom_Components:SW_Tactile_SKHH_Angled
Connections:
- net GP_17 is gone; now on net GP_4: R27.2
- net +3V3: now also J15.2 (VCC)
- net +5V_IN: now also J13.1 (Pin_1), NT8.2; no longer D1.1 (K)
- net +5V_RAW: now also D1.1 (K), J13.2 (Pin_2), J14.1 (Pin_1), J16.2 (Pin_2), NT8.1; no longer D1.2 (A)
- net +5V_VOUT: now also J13.3 (Pin_3)
- net GND: now also J2B1.10, J2B1.5, J2B1.6, J2B1.7, J2B1.8, J2B1.SH, J12.1 (GND), J12.6 (SH), J15.1 (GND), J16.1 (Pin_1)
- net GP_2: now also U1.4 (GP2), J15.5 (SCK); no longer R28.2
- net GP_26: now also U1.31 (GP26)
- net GP_27: now also U1.32 (GP27)
- net GP_28: now also U1.34 (GP28)
- net VGA_B: now also J2B1.3
- net VGA_G: now also J2B1.2
- net VGA_HS: now also J2B1.13
- net VGA_R: now also J2B1.1
- net VGA_VS: now also J2B1.14
- net GP_3: now reaches U1.5 (GP3)
- net GP_3: now also J15.4 (MOSI)
- net GP_4: now reaches U1.6 (GP4)
- net GP_4: now also J15.3 (MISO)
- net GP_5: now reaches U1.7 (GP5)
- net GP_5: now also R28.2, J15.6 (CS)
- new net: D1.2 (A), J12.5 (VBUS), J14.2 (Pin_2)
- no-connect marks 41 -> 26
Other:
- moved on the sheet: C19, J1, J2, J2B1
