File: schematics/rp2040_black_vga/rp2040_black_vga.kicad_pcb (KiCad board)
At the start: 2 copper layers, 13 x 1.4 mm, 65 parts, among them J1 Jack-DC, J10 Conn_01x02, J13 Conn_01x03, J14 Conn_01x02, J16 Conn_01x02, J2 Conn_01x02, J2B1 DE15_Socket, J4 Mini-DIN-6, J5 Conn_02x20_Odd_Even, J6 DE9_Pins, J7 DE9_Pins, J8 Audio OUT, J8B1 OUT_A, J9 Audio IN, J9B1 IN_A, Q1 S9014, Q2 S9014, SW1 RESET, U1 YD-RP2040 TypeC Black Clone

Commit message: pictures
Parts:
- moved Q1 5.16 mm to (162.6, 106.7), turned to 90 degrees
- moved Q2 5.16 mm to (167.6, 96.5), turned to 90 degrees
